File: Power.kicad_sch (KiCad schematic)
At the start: 61 parts, among them J4 On/Off, U1 AMS1117-3.3, U2 DRV8301, U3 TP2604-SR

Commit message: Added Gerber Files
Parts:
- NT1: footprint (none) -> Additions:NT3_Small
