File: STM32F4 64LQFP.kicad_sch (KiCad schematic)
At the start: 16 parts, among them J1 UNUSED MCU PINS, P5 SWD, U5 STM32F405RGT6, X1 8MHz 10ppm (X50328MSB2GI)

Commit message: Added Gerber Files
Parts:
- removed J1: UNUSED MCU PINS, Connector_PinHeader_2.00mm:PinHeader_2x05_P2.00mm_Vertical, symbol Connector_Generic:Conn_02x05_Top_Bottom
Connections:
- net PB12: no longer names the net of U5.33 (PB12)
- net PB3: no longer names the net of U5.55 (PB3(JTDO/TRACESWO))
- net PB4: no longer names the net of U5.56 (PB4(NJTRST))
- net PC13: no longer names the net of U5.2 (PC13_(RTC_AF1))
- net PC14: no longer names the net of U5.3 (PC14-OSC32_IN)
- net PC15: no longer names the net of U5.4 (PC15-OSC32_OUT)
- net PC5: no longer names the net of U5.25 (PC5(ADC12_IN15))
- net PD2: no longer names the net of U5.54 (PD2)
- no-connect marks 2 -> 10
Other:
- note removed: "Unused MCU Pins"
