File: Stupid_FOCer.kicad_sch (KiCad schematic)
At the start: 52 parts, among them J2 Conn_01x07, J3 Conn_01x03, J6 Conn_01x03, J7 Conn_01x03, P1 MOTOR1, P2 MOTOR1, P3 MOTOR1, P4 HALL/Encoder, P6 USB_C_Plug_USB2.0

Commit message: Added Gerber Files
Parts:
- removed H2, H6, H8: MountingHole, MountingHole:MountingHole_3.2mm_M3_ISO14580_Pad, symbol Mechanical:MountingHole
- removed H7: MountingHole, MountingHole:MountingHole_3.2mm_M3_ISO14580_Pad, symbol Mechanical:MountingHole_Pad
- removed NEG3: MOTOR3, CRF1:1pin_4mm, symbol BLDC_4-rescue:CONN_1
- removed P1, P2, P3: MOTOR1, CRF1:1pin_4mm, symbol BLDC_4-rescue:CONN_1
- added J5: Conn_01x08, Connector_PinSocket_2.54mm:PinSocket_1x08_P2.54mm_Vertical, symbol Connector_Generic:Conn_01x08
- added POS2: POS, Additions:MountingPad, symbol BLDC_4-rescue:CONN_1
- added R69: DNP, Resistor_SMD:R_0603_1608Metric, symbol BLDC_4-rescue:R-RESCUE-BLDC_4
- H1, H13, H5: footprint MountingHole:MountingHole_3.2mm_M3_ISO14580_Pad -> MountingHole:MountingHole_3.2mm_M3_ISO14580
- NT2: footprint (none) -> NetTie:NetTie-3_SMD_Pad0.5mm
- POS1: footprint CRF1:1pin_4mm -> Additions:MountingPad
Connections:
- net GND: now also J5.2 (Pin_2), J5.7 (Pin_7), POS2.1
- net RX_SDA_IN: now also J5.5 (Pin_5)
- net TX_SCL_MOSI_IN: now also J5.6 (Pin_6)
- net VCC: now also J5.4 (Pin_4), R69.1
- new net: J5.1 (Pin_1), R69.2
- no-connect marks 3 -> 5
Other:
- sheet Power MOSFETS ports: added none; removed PHASE_1, PHASE_2, PHASE_3
- moved on the sheet: H13, NT2
