File: mosfets.kicad_sch (KiCad schematic)
At the start: 53 parts, among them Q1 NCEP60T20, Q2 NCEP60T20, Q3 NCEP60T20, Q4 NCEP60T20, Q5 NCEP60T20, Q6 NCEP60T20

Commit message: Added Gerber Files
Parts:
- removed NT3, NT4, NT5: NetTie_2, symbol Device:NetTie_2
- added P1, P2, P3: MOTOR1, Additions:MountingPad, symbol BLDC_4-rescue:CONN_1
- NT10, NT11, NT6, NT7, NT8, NT9: footprint (none) -> NetTie:NetTie-2_SMD_Pad0.5mm
- R? (x6): value 10R -> 20R
Connections:
- net H1_VS: now also P1.1
- net H2_VS: now also P2.1
- net H3_VS: now also P3.1
